Commit message: inverse kinematics for 3 dof robot

File: urdf/robot.urdf (robot description, URDF)
Before this commit: robot 3dof_robot, 11 links, 10 joints
Joints:
- joint link_1_to_link_2: limit lower=-1.57 upper=1.57 effort=50 velocity=1.0 -> lower=-3.14 upper=3.14 effort=50 velocity=1.0
- joint link_2_to_link_3: limit lower=-1.57 upper=1.57 effort=50 velocity=1.0 -> lower=-3.14 upper=3.14 effort=50 velocity=1.0
- joint link_3_to_link_4: limit lower=-1.57 upper=1.57 effort=50 velocity=1.0 -> lower=-3.14 upper=3.14 effort=50 velocity=1.0
- joint link_4_to_gripper: limit lower=-1.57 upper=1.57 effort=50 velocity=1.0 -> lower=-3.14 upper=3.14 effort=50 velocity=1.0

File: urdf/robot.urdf.xacro (robot description, xacro)
@@ -108,5 +108,5 @@
     <origin xyz="0 0 ${l1}" rpy="0 0 0"/>
     <axis xyz="0 1 0"/>
-    <limit lower="-1.57" upper="1.57" effort="50" velocity="1.0"/>
+    <limit lower="-3.14" upper="3.14" effort="50" velocity="1.0"/>
   </joint>
   <link name="joint_1_visual">
@@ -125,5 +125,5 @@
     <origin xyz="0 0 ${l2}" rpy="0 0 0"/>
     <axis xyz="0 1 0"/>
-    <limit lower="-1.57" upper="1.57" effort="50" velocity="1.0"/>
+    <limit lower="-3.14" upper="3.14" effort="50" velocity="1.0"/>
   </joint>
   <link name="joint_2_visual">
@@ -142,5 +142,5 @@
     <origin xyz="0 0 ${l3}" rpy="0 0 0"/>
     <axis xyz="0 1 0"/>
-    <limit lower="-1.57" upper="1.57" effort="50" velocity="1.0"/>
+    <limit lower="-3.14" upper="3.14" effort="50" velocity="1.0"/>
   </joint>
   <link name="joint_3_visual">
@@ -205,5 +205,5 @@
     <origin xyz="0 0 ${l4}" rpy="0 0 0"/>
     <axis xyz="0 1 0"/>
-    <limit lower="-1.57" upper="1.57" effort="50" velocity="1.0"/>
+    <limit lower="-3.14" upper="3.14" effort="50" velocity="1.0"/>
   </joint>
   <link name="joint_4_visual">
